Commit message: Add files via upload

File: urdf_models/L6V3.1_left/linkerhand_L6V3.1_left.urdf (robot description, URDF)
Before this commit: robot linkerhand_L6V3.1_left_1.9, 12 links, 11 joints
Joints:
- joint index_dip: origin xyz=0.001001 -0.000537 0.028003 rpy=0 0 0 -> xyz=0.00093749 0 0.028002 rpy=0 0 0
- joint middle_dip: origin xyz=0.000994 0.000058 0.028008 rpy=0 0 0 -> xyz=0.00093749 0 0.028002 rpy=0 0 0
- joint pinky_dip: origin xyz=0.000979 0.001534 0.027967 rpy=0 0 0 -> xyz=0.00093749 0 0.028002 rpy=0 0 0
- joint ring_dip: origin xyz=0.000979 0.001534 0.027967 rpy=0 0 0 -> xyz=0.00093749 0 0.028002 rpy=0 0 0
